File: clock_module/clock_module.kicad_sch (KiCad schematic)
At the start: 0 parts

Commit message: pcb routes (unfinished)
Parts:
- added H1, H2, H3, H4: MountingHole, MountingHole:MountingHole_3.2mm_M3, symbol Mechanical:MountingHole
Other:
- note added: "Mounting Holes"

Commit message: finished board
Other:
- title: (none) -> Clock Module
Changed lines of the file:
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@@
 	(generator_version "9.0")
 	(paper "A4")
+	(title_block
+		(title "Clock Module")
+		(date "2026-05-26")
+		(rev "Gustavo C. S.")
+	)
 	(text "Mounting Holes"
 		(exclude_from_sim no)
