File: clock_module/clock_module.kicad_pcb (KiCad board)
At the start: 4 copper layers, 70 x 34 mm, 41 parts, among them J1 Connector, USB-TYPE-C-16P, J2 Conn_01x03, SW1 SW_SPDT, U1 USBLC6-2SC6, U2 NE555DR, U3 NE555DR, U4 74HC08D, U5 74HC32D, U6 NE555DR, U7 74HC04D

Commit message: finished board
Parts:
- moved J2 0.47 mm to (154.4, 66.5)
Routing:
- net /Main Circuit/CLK_SIGNAL: track 11.7 -> 45.3 mm, vias 2 -> 4
- net /Main Circuit/HLT: track 0.00 -> 33.2 mm, vias 0 -> 2
- net /Main Circuit/!CLK_SIGNAL: track 0.00 -> 32.2 mm
- net /Main Circuit/!SIG_SELECT: track 0.00 -> 28.3 mm, vias 0 -> 2
- net Net-(U4-2Y): track 0.00 -> 25.7 mm, vias 0 -> 2
- net Net-(U4-1Y): track 0.00 -> 25.5 mm, vias 0 -> 2
- net Net-(U4-3A): track 0.00 -> 17.2 mm, vias 0 -> 2
- net Net-(U4-3B): track 0.00 -> 10.9 mm, vias 0 -> 2
- net +5V: track 158.1 -> 161.4 mm
- net /Main Circuit/SIG_SELECT: track 43.0 -> 44.7 mm
- net GND: track 34.4 -> 33.6 mm, vias 37 -> 27
Other:
- board text added: "!CLK"
- board text added: "CLK"
- board text added: "Clock Module"
- board text added: "HLT"
- board text added: "JLCJLCJLCJLC"
- board text added: "Made by: Gustavo Caetano da Silva Version: v1.0.0"

Commit message: final v1.0.0 project
Parts:
- removed J2: Conn_01x03, Connector_PinHeader_2.54mm:PinHeader_1x03_P2.54mm_Vertical
- added J3: Conn_01x05, Connector_PinHeader_2.54mm:PinHeader_1x05_P2.54mm_Vertical, F.Cu at (155.0, 70.8)
- R6: value 1kΩ -> 200kΩ
- RV1: value 1M -> 200k
- moved R6 0.21 mm to (123.4, 81.4)
Routing:
- net +5V: track 161.4 -> 177.5 mm
- net /Main Circuit/HLT: track 33.2 -> 35.6 mm
- net /Main Circuit/!CLK_SIGNAL: track 32.2 -> 33.9 mm
- net Net-(U4-1Y): track 25.5 -> 23.8 mm
- net /Main Circuit/CLK_SIGNAL: track 45.3 -> 46.4 mm, vias 4 -> 6
- net /Main Circuit/!SIG_SELECT: track 28.3 -> 29.0 mm
Other:
- board text added: "+5V"
- board text added: "GND"
